File: pcb/PCB.kicad_pcb (KiCad board)
At the start: 4 copper layers, 100 x 60 mm, 33 parts, among them J1 TE 770966-2, J2 TE 770966-2, J3 JST B04B-XASK, K1 AZDC6, Q1 IRLZ44N, U1 LM339, U2 LTV-817S, U3 VRB1205YMD-15WR3

Commit message: update pcb too
Connections:
- U1 pad 4: Net-(D2-A2) -> Net-(D1-A2)
- U1 pad 5: Net-(D1-A2) -> Net-(D2-A2)
Routing:
- net Net-(D1-A2): track 23.0 -> 25.9 mm
Changed lines of the file:
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@@
       (net 1 "+5V") (pinfunction "V+") (pintype "power_in"))
     (pad "4" smd roundrect (at -2.8625 0 180) (size 1.475 0.4) (layers "B.Cu" "B.Paste" "B.Mask") (roundrect_rratio 0.25)
-      (net 4 "Net-(D2-A2)") (pinfunction "-") (pintype "input"))
+      (net 3 "Net-(D1-A2)") (pinfunction "-") (pintype "input"))
     (pad "5" smd roundrect (at -2.8625 -0.65 180) (size 1.475 0.4) (layers "B.Cu" "B.Paste" "B.Mask") (roundrect_rratio 0.25)
-      (net 3 "Net-(D1-A2)") (pinfunction "+") (pintype "input"))
+      (net 4 "Net-(D2-A2)") (pinfunction "+") (pintype "input"))
     (pad "6" smd roundrect (at -2.8625 -1.3 180) (size 1.475 0.4) (layers "B.Cu" "B.Paste" "B.Mask") (roundrect_rratio 0.25))
     (pad "7" smd roundrect (at -2.8625 -1.95 180) (size 1.475 0.4) (layers "B.Cu" "B.Paste" "B.Mask") (roundrect_rratio 0.25))
@@
   (segment (start 75.34 75.34) (end 80 80) (width 1) (layer "B.Cu") (net 2))
   (segment (start 89.425 90) (end 89.5 90) (width 1) (layer "B.Cu") (net 3))
-  (segment (start 106.125001 89.65) (end 102.775001 93) (width 0.25) (layer "B.Cu") (net 3))
+  (segment (start 100 93) (end 95.5 88.5) (width 0.25) (layer "B.Cu") (net 3))
+  (segment (start 108.25 89.650001) (end 108.25 90.833102) (width 0.25) (layer "B.Cu") (net 3))
+  (segment (start 108.25 90.833102) (end 106.083102 93) (width 0.25) (layer "B.Cu") (net 3))
+  (segment (start 106.083102 93) (end 100 93) (width 0.25) (layer "B.Cu") (net 3))
   (segment (start 92 87.5) (end 94.5 87.5) (width 1) (layer "B.Cu") (net 3))
-  (segment (start 98.5 93) (end 95.5 90) (width 0.25) (layer "B.Cu") (net 3))
   (segment (start 89.5 90) (end 92 87.5) (width 1) (layer "B.Cu") (net 3))
-  (segment (start 102.775001 93) (end 98.5 93) (width 0.25) (layer "B.Cu") (net 3))
-  (segment (start 106.8625 89.65) (end 106.125001 89.65) (width 0.25) (layer "B.Cu") (net 3))
-  (segment (start 95.5 90) (end 95.5 88.5) (width 0.25) (layer "B.Cu") (net 3))
+  (segment (start 107.599999 89) (end 108.25 89.650001) (width 0.25) (layer "B.Cu") (net 3))
+  (segment (start 106.8625 89) (end 107.599999 89) (width 0.25) (layer "B.Cu") (net 3))
   (segment (start 94.5 87.5) (end 95.5 88.5) (width 1) (layer "B.Cu") (net 3))
   (segment (start 94.5 73.5) (end 95.5 72.5) (width 1) (layer "B.Cu") (net 4))
-  (segment (start 106.8625 89) (end 105 89) (width 0.25) (layer "B.Cu") (net 4))
+  (segment (start 103.95 87.95) (end 105.65 89.65) (width 0.25) (layer "B.Cu") (net 4))
   (segment (start 91.9625 73.5) (end 89.4625 71) (width 1) (layer "B.Cu") (net 4))
-  (segment (start 100 72.5) (end 95.5 72.5) (width 0.25) (layer "B.Cu") (net 4))
-  (segment (start 103.95 76.45) (end 100 72.5) (width 0.25) (layer "B.Cu") (net 4))
+  (segment (start 103.95 76.45) (end 103.95 87.95) (width 0.25) (layer "B.Cu") (net 4))
   (segment (start 92 73.5) (end 94.5 73.5) (width 1) (layer "B.Cu") (net 4))
+  (segment (start 95.5 72.5) (end 100 72.5) (width 0.25) (layer "B.Cu") (net 4))
   (segment (start 92 73.5) (end 91.9625 73.5) (width 1) (layer "B.Cu") (net 4))
-  (segment (start 103.95 87.95) (end 103.95 76.45) (width 0.25) (layer "B.Cu") (net 4))
-  (segment (start 105 89) (end 103.95 87.95) (width 0.25) (layer "B.Cu") (net 4))
+  (segment (start 100 72.5) (end 103.95 76.45) (width 0.25) (layer "B.Cu") (net 4))
+  (segment (start 105.65 89.65) (end 106.8625 89.65) (width 0.25) (layer "B.Cu") (net 4))
   (segment (start 75.34 65.66) (end 84 57) (width 1) (layer "B.Cu") (net 5))
   (segment (start 75.34 70.93) (end 75.34 65.66) (width 1) (layer "B.Cu") (net 5))
